File: pcb project/deep blue delay/deep blue delay.kicad_pcb (KiCad board)
At the start: 2 copper layers, 55 x 65 mm, 62 parts, among them J1 in-outs, J2 shorter delay, J3 AGND-DGND, J4 LED-OMIT, U1 OP275, U2 L78L05_SOT89, U3 PT2399

Commit message: ss
Other:
- net class Default removed
